Commit message: Your commit message

File: install/arduinobot_description/share/arduinobot_description/urdf/arduinobot.urdf.xacro (robot description, xacro)
@@ -1 +1,15 @@
-/home/farr97/arduinobot_ws/src/arduinobot_description/urdf/arduinobot.urdf.xacro
+<?xml version="1.0"?>
+<robot xmlns:xacro="http://www.ros.org/wiki/xacro" name="arduinobot">
+    <xacro:arg name="use_gazebo" default="false"/>
+    <!-- Include properties first -->
+    <xacro:include filename="$(find arduinobot_description)/urdf/properties.xacro"/>
+    <!-- Import robot parts -->
+    <xacro:include filename="$(find arduinobot_description)/urdf/base_and_base_plate.xacro"/>
+    <xacro:include filename="$(find arduinobot_description)/urdf/arms.xacro"/>
+    <xacro:include filename="$(find arduinobot_description)/urdf/connectors.xacro"/>
+    <xacro:include filename="$(find arduinobot_description)/urdf/grippers.xacro"/>
+    <!-- Import Gazebo elements if needed -->
+    <xacro:if value="$(arg use_gazebo)">
+        <xacro:include filename="$(find arduinobot_description)/urdf/arduinobot_gazebo.xacro"/>
+    </xacro:if>
+</robot>

File: install/arduinobot_description/share/arduinobot_description/urdf/arduinobot_gazebo.xacro (robot description, xacro)
@@ -1 +1,38 @@
-/home/farr97/arduinobot_ws/src/arduinobot_description/urdf/arduinobot_gazebo.xacro
+<?xml version="1.0"?>
+<robot xmlns:xacro="http://www.ros.org/wiki/xacro">
+    <!-- Gazebo Colors -->
+    <gazebo reference="base_link">
+        <material>Gazebo/Grey</material>
+    </gazebo>
+    <gazebo reference="base_plate">
+        <material>Gazebo/Blue</material>
+    </gazebo>
+    <gazebo reference="arm_1">
+        <material>Gazebo/Grey</material>
+    </gazebo>
+    <gazebo reference="arm_2">
+        <material>Gazebo/Grey</material>
+    </gazebo>
+    <gazebo reference="arm_3">
+        <material>Gazebo/Grey</material>
+    </gazebo>
+    <gazebo reference="inner_circle">
+        <material>Gazebo/Grey</material>
+    </gazebo>
+    <gazebo reference="gripper_1">
+        <material>Gazebo/Grey</material>
+    </gazebo>
+    <gazebo reference="gripper_2">
+        <material>Gazebo/Grey</material>
+    </gazebo>
+    <gazebo reference="gripper_3">
+        <material>Gazebo/Grey</material>
+    </gazebo>
+    <!-- Gazebo plugins -->
+    <gazebo>
+        <plugin name="gazebo_ros_control" filename="libgazebo_ros_control.so">
+            <robotNamespace>/arduinobot</robotNamespace>
+            <robotSimType>gazebo_ros_control/DefaultRobotHWSim</robotSimType>
+        </plugin>
+    </gazebo>
+</robot>

File: install/arduinobot_description/share/arduinobot_description/urdf/arduinobot_ros2_control.xacro (robot description, xacro)
@@ -1 +1,71 @@
-/home/farr97/arduinobot_ws/src/arduinobot_description/urdf/arduinobot_ros2_control.xacro
+<?xml version="1.0"?>
+<robot xmlns:xacro="http://www.ros.org/wiki/xacro">
+    <xacro:arg name="is_ignition" default="true"/>
+    <ros2_control name="RobotSystem" type="system">
+        <xacro:property name="PI" value="3.141592653589793"/>
+        <xacro:property name="PI_2" value="${PI / 2.0}"/>
+        <!-- Gazebo system plugin -->
+        <xacro:property name="system" value="ros_gz_sim"/>
+        <xacro:if value="$(arg is_ignition)">
+            <hardware>
+                <plugin>ign_ros2_control/IgnitionSystem</plugin>
+            </hardware>
+        </xacro:if>
+        <xacro:unless value="$(arg is_ignition)">
+            <hardware>
+                <plugin>arduinobot_controller/ArduinobotInterface</plugin>
+                <param name="serial_port">/dev/ttyACM0</param>
+            </hardware>
+        </xacro:unless>
+        <!-- Base plate joint -->
+        <joint name="base_to_base_plate">
+            <command_interface name="position">
+                <param name="min">-${PI_2}</param>
+                <param name="max">${PI_2}</param>
+            </command_interface>
+            <state_interface name="position"/>
+            <state_interface name="velocity"/>
+        </joint>
+        <!-- Arm joints -->
+        <joint name="base_plate_to_arm_1">
+            <command_interface name="position">
+                <param name="min">-${PI_2}</param>
+                <param name="max">${PI_2}</param>
+            </command_interface>
+            <state_interface name="position"/>
+            <state_interface name="velocity"/>
+        </joint>
+        <joint name="arm_1_to_arm_2">
+            <command_interface name="position">
+                <param name="min">-${PI_2}</param>
+                <param name="max">${PI_2}</param>
+            </command_interface>
+            <state_interface name="position"/>
+            <state_interface name="velocity"/>
+        </joint>
+        <joint name="arm_2_to_inner_circle">
+            <command_interface name="position">
+                <param name="min">-${PI}</param>
+                <param name="max">0.0</param>
+            </command_interface>
+            <state_interface name="position"/>
+            <state_interface name="velocity"/>
+        </joint>
+        <joint name="arm_2_to_arm_3">
+            <command_interface name="position">
+                <param name="min">-${PI_2}</param>
+                <param name="max">${PI_2}</param>
+            </command_interface>
+            <state_interface name="position"/>
+            <state_interface name="velocity"/>
+        </joint>
+    </ros2_control>
+    <!-- Gazebo ros2_control plugin -->
+    <gazebo>
+        <plugin filename="libgz_sim_ros2_control-system.so"
+                name="gz_sim_ros2_control">
+            <parameters>$(find arduinobot_description)/config/ros2_controllers.yaml</parameters>
+            <robot_param_node>robot_state_publisher</robot_param_node>
+        </plugin>
+    </gazebo>
+</robot>

File: install/arduinobot_description/share/arduinobot_description/urdf/arms.xacro (robot description, xacro)
@@ -1 +1,104 @@
-/home/farr97/arduinobot_ws/src/arduinobot_description/urdf/arms.xacro
+<?xml version="1.0"?>
+<robot xmlns:xacro="http://www.ros.org/wiki/xacro">
+    <!-- Include properties file -->
+    <xacro:include filename="$(find arduinobot_description)/urdf/properties.xacro"/>
+    <!-- Arm 1 -->
+    <link name="arm_1">
+        <visual>
+            <origin rpy="0 0 0" xyz="0 0 0"/>
+            <geometry>
+                <mesh filename="package://arduinobot_description/meshes/arm_1.dae" scale="5 5 5"/>
+            </geometry>
+            <material name="grey">
+                <color rgba="0.7 0.7 0.7 1.0"/>
+            </material>
+        </visual>
+        <collision>
+            <origin rpy="0 0 0" xyz="0 0 0"/>
+            <geometry>
+                <box size="0.03 0.03 0.15"/>
+            </geometry>
+        </collision>
+        <inertial>
+            <origin xyz="0 0 0" rpy="0 0 0"/>
+            <mass value="0.25"/>
+            <inertia ixx="0.0003" ixy="0.0" ixz="0.0"
+                    iyy="0.0003" iyz="0.0"
+                    izz="0.00001"/>
+        </inertial>
+    </link>
+    <joint name="base_plate_to_arm_1" type="revolute">
+        <parent link="base_plate"/>
+        <child link="arm_1"/>
+        <origin rpy="0 0 0" xyz="0 0 0.0012"/>
+        <axis xyz="0 1 0"/>
+        <limit lower="-${PI/3}" upper="${PI/3}" effort="${effort}" velocity="${velocity}"/>
+        <dynamics damping="0.5" friction="0.1"/>
+    </joint>
+    <!-- Arm 2 -->
+    <link name="arm_2">
+        <visual>
+            <origin rpy="0 0 0" xyz="0 0 0"/>
+            <geometry>
+                <mesh filename="package://arduinobot_description/meshes/arm_2.dae" scale="5 5 5"/>
+            </geometry>
+            <material name="grey">
+                <color rgba="0.7 0.7 0.7 1.0"/>
+            </material>
+        </visual>
+        <collision>
+            <origin rpy="0 0 0" xyz="0 0 0"/>
+            <geometry>
+                <box size="0.03 0.03 0.15"/>
+            </geometry>
+        </collision>
+        <inertial>
+            <origin xyz="0 0 0" rpy="0 0 0"/>
+            <mass value="0.2"/>
+            <inertia ixx="0.0002" ixy="0.0" ixz="0.0"
+                    iyy="0.0002" iyz="0.0"
+                    izz="0.00001"/>
+        </inertial>
+    </link>
+    <joint name="arm_1_to_arm_2" type="revolute">
+        <parent link="arm_1"/>
+        <child link="arm_2"/>
+        <origin rpy="0 0 0" xyz="0 0 0.035"/>
+        <axis xyz="0 1 0"/>
+        <limit lower="-${PI/3}" upper="${PI/3}" effort="${effort}" velocity="${velocity}"/>
+        <dynamics damping="0.5" friction="0.1"/>
+    </joint>
+    <!-- Arm 3 -->
+    <link name="arm_3">
+        <visual>
+            <origin rpy="0 0 0" xyz="0 0 0"/>
+            <geometry>
+                <mesh filename="package://arduinobot_description/meshes/arm_3.dae" scale="5 5 5"/>
+            </geometry>
+            <material name="grey">
+                <color rgba="0.7 0.7 0.7 1.0"/>
+            </material>
+        </visual>
+        <collision>
+            <origin rpy="0 0 0" xyz="0 0 0"/>
+            <geometry>
+                <box size="0.03 0.03 0.15"/>
+            </geometry>
+        </collision>
+        <inertial>
+            <origin xyz="0 0 0" rpy="0 0 0"/>
+            <mass value="0.15"/>
+            <inertia ixx="0.0002" ixy="0.0" ixz="0.0"
+                    iyy="0.0002" iyz="0.0"
+                    izz="0.00001"/>
+        </inertial>
+    </link>
+    <joint name="arm_2_to_arm_3" type="revolute">
+        <parent link="arm_2"/>
+        <child link="arm_3"/>
+        <origin rpy="0 0 0" xyz="0 0 0.035"/>
+        <axis xyz="0 1 0"/>
+        <limit lower="-${PI_2}" upper="${PI_2}" effort="${effort}" velocity="${velocity}"/>
+        <dynamics damping="0.5" friction="0.1"/>
+    </joint>
+</robot>

File: install/arduinobot_description/share/arduinobot_description/urdf/base_and_base_plate.xacro (robot description, xacro)
@@ -1 +1,67 @@
-/home/farr97/arduinobot_ws/src/arduinobot_description/urdf/base_and_base_plate.xacro
+<?xml version="1.0"?>
+<robot xmlns:xacro="http://www.ros.org/wiki/xacro" name="arduinobot">
+    <link name="world"/>
+    <!-- Base Link -->
+    <link name="base_link">
+        <visual>
+            <origin rpy="0 0 0" xyz="0 0 0"/>
+            <geometry>
+                <mesh filename="package://arduinobot_description/meshes/basement_1.dae" scale="5 5 5"/>
+            </geometry>
+            <material name="dark_grey">
+                <color rgba="0.3 0.3 0.3 1.0"/>
+            </material>
+        </visual>
+        <collision>
+            <origin rpy="0 0 0" xyz="0 0 0"/>
+            <geometry>
+                <cylinder radius="0.06" length="0.04"/>
+            </geometry>
+        </collision>
+        <inertial>
+            <origin xyz="0 0 0.02" rpy="0 0 0"/>
+            <mass value="0.5"/>
+            <inertia ixx="0.00015" ixy="0.0" ixz="0.0"
+                    iyy="0.00015" iyz="0.0"
+                    izz="0.00025"/>
+        </inertial>
+    </link>
+    <joint name="virtual_joint" type="fixed">
+        <parent link="world"/>
+        <child link="base_link"/>
+        <origin rpy="0 0 0" xyz="0 0 0"/>
+    </joint>
+    <!-- Base Plate -->
+    <link name="base_plate">
+        <visual>
+            <origin rpy="0 0 0" xyz="0 0 0"/>
+            <geometry>
+                <mesh filename="package://arduinobot_description/meshes/base_plate_2.dae" scale="5 5 5"/>
+            </geometry>
+            <material name="blue">
+                <color rgba="0.2 0.2 0.8 1.0"/>
+            </material>
+        </visual>
+        <collision>
+            <origin rpy="0 0 0" xyz="0 0 0"/>
+            <geometry>
+                <cylinder radius="0.04" length="0.04"/>
+            </geometry>
+        </collision>
+        <inertial>
+            <origin xyz="0 0 0" rpy="0 0 0"/>
+            <mass value="0.3"/>
+            <inertia ixx="0.0001" ixy="0.0" ixz="0.0"
+                    iyy="0.0001" iyz="0.0"
+                    izz="0.00015"/>
+        </inertial>
+    </link>
+    <joint name="base_to_base_plate" type="revolute">
+        <parent link="base_link"/>
+        <child link="base_plate"/>
+        <origin rpy="0 0 0" xyz="0 0 0.009"/>
+        <axis xyz="0 0 1"/>
+        <limit lower="-${PI_2}" upper="${PI_2}" effort="${effort}" velocity="${velocity}"/>
+        <dynamics damping="0.5" friction="0.1"/>
+    </joint>
+</robot>

File: install/arduinobot_description/share/arduinobot_description/urdf/camera.xacro (robot description, xacro)
@@ -1 +1,32 @@
-/home/farr97/arduinobot_ws/src/arduinobot_description/urdf/camera.xacro
+<?xml version="1.0"?>
+<robot xmlns:xacro="http://ros.org/wiki/xacro">
+<!-- Camera Link -->
+<link name="camera_link">
+    <visual>
+        <origin rpy="0 0 0" xyz="0 0 0.025"/>
+        <geometry>
+            <box size="0.025 0.025 0.025"/>
+        </geometry>
+        <material name="black">
+            <color rgba="0.1 0.1 0.1 1.0"/>
+        </material>
+    </visual>
+    <collision>
+        <origin rpy="0 0 0" xyz="0 0 0.025"/>
+        <geometry>
+            <box size="0.025 0.025 0.025"/>
+        </geometry>
+    </collision>
+    <inertial>
+        <origin xyz="0 0 0.025" rpy="0 0 0"/>
+        <mass value="0.1"/>
+        <inertia ixx="0.0001" ixy="0.0" ixz="0.0" iyy="0.0001" iyz="0.0" izz="0.0001"/>
+    </inertial>
+</link>
+<!-- Joint to Attach Camera to Base -->
+<joint name="base_to_camera" type="fixed">
+    <parent link="base_link"/>
+    <child link="camera_link"/>
+    <origin xyz="0.15 0 0.1" rpy="0 0.7 0"/>
+</joint>
+</robot>

File: install/arduinobot_description/share/arduinobot_description/urdf/connectors.xacro (robot description, xacro)
@@ -1 +1,36 @@
-/home/farr97/arduinobot_ws/src/arduinobot_description/urdf/connectors.xacro
+<?xml version="1.0"?>
+<robot xmlns:xacro="http://ros.org/wiki/xacro">
+    <!-- inner_circle -->
+    <link name="inner_circle">
+        <visual>
+            <origin rpy="0 0 0" xyz="0 0 0"/>
+            <geometry>
+                <mesh filename="package://arduinobot_description/meshes/inner_circle.dae" scale="5 5 5"/>
+            </geometry>
+            <material name="grey">
+                <color rgba="0.7 0.7 0.7 1.0"/>
+            </material>
+        </visual>
+        <collision>
+            <origin rpy="0 0 0" xyz="0 0 0"/>
+            <geometry>
+                <cylinder radius="0.025" length="0.03"/>
+            </geometry>
+        </collision>
+        <inertial>
+            <origin xyz="0 0 0" rpy="0 0 0"/>
+            <mass value="0.1"/>
+            <inertia ixx="0.00001" ixy="0.0" ixz="0.0"
+                    iyy="0.00001" iyz="0.0"
+                    izz="0.00001"/>
+        </inertial>
+    </link>
+    <joint name="arm_2_to_inner_circle" type="revolute">
+        <parent link="arm_2"/>
+        <child link="inner_circle"/>
+        <origin rpy="0 0 0" xyz="-0.16 -0.01 0.21"/>
+        <axis xyz="1 0 0"/>
+        <limit lower="-${PI}" upper="0.0" effort="${effort}" velocity="${velocity}"/>
+        <dynamics damping="0.5" friction="0.1"/>
+    </joint>
+</robot>

File: install/arduinobot_description/share/arduinobot_description/urdf/grippers.xacro (robot description, xacro)
@@ -1 +1,100 @@
-/home/farr97/arduinobot_ws/src/arduinobot_description/urdf/grippers.xacro
+<?xml version="1.0"?>
+<robot xmlns:xacro="http://www.ros.org/wiki/xacro">
+    <!-- Gripper Links -->
+    <link name="gripper_1">
+        <visual>
+            <origin rpy="0 0 0" xyz="0 0 0"/>
+            <geometry>
+                <mesh filename="package://arduinobot_description/meshes/gripper_1.dae" scale="5 5 5"/>
+            </geometry>
+            <material name="grey">
+                <color rgba="0.7 0.7 0.7 1.0"/>
+            </material>
+        </visual>
+        <collision>
+            <origin rpy="0 0 0" xyz="0 0 0"/>
+            <geometry>
+                <box size="0.02 0.04 0.02"/>
+            </geometry>
+        </collision>
+        <inertial>
+            <origin xyz="0 0 0" rpy="0 0 0"/>
+            <mass value="0.05"/>
+            <inertia ixx="0.00001" ixy="0.0" ixz="0.0"
+                    iyy="0.00002" iyz="0.0"
+                    izz="0.00001"/>
+        </inertial>
+    </link>
+    <link name="gripper_2">
+        <visual>
+            <origin rpy="0 0 0" xyz="0 0 0"/>
+            <geometry>
+                <mesh filename="package://arduinobot_description/meshes/gripper_2.dae" scale="5 5 5"/>
+            </geometry>
+            <material name="grey"/>
+        </visual>
+        <collision>
+            <origin rpy="0 0 0" xyz="0 0 0"/>
+            <geometry>
+                <box size="0.02 0.04 0.02"/>
+            </geometry>
+        </collision>
+        <inertial>
+            <origin xyz="0 0 0" rpy="0 0 0"/>
+            <mass value="0.05"/>
+            <inertia ixx="0.00001" ixy="0.0" ixz="0.0"
+                    iyy="0.00002" iyz="0.0"
+                    izz="0.00001"/>
+        </inertial>
+    </link>
+    <link name="gripper_3">
+        <visual>
+            <origin rpy="0 0 0" xyz="0 0 0"/>
+            <geometry>
+                <mesh filename="package://arduinobot_description/meshes/gripper_3.dae" scale="5 5 5"/>
+            </geometry>
+            <material name="grey"/>
+        </visual>
+        <collision>
+            <origin rpy="0 0 0" xyz="0 0 0"/>
+            <geometry>
+                <box size="0.02 0.04 0.02"/>
+            </geometry>
+        </collision>
+        <inertial>
+            <origin xyz="0 0 0" rpy="0 0 0"/>
+            <mass value="0.05"/>
+            <inertia ixx="0.00001" ixy="0.0" ixz="0.0"
+                    iyy="0.00002" iyz="0.0"
+                    izz="0.00001"/>
+        </inertial>
+    </link>
+    <!-- Gripper Joints -->
+    <joint name="inner_circle_to_gripper_1" type="revolute">
+        <parent link="inner_circle"/>
+        <child link="gripper_1"/>
+        <origin rpy="0 0 0" xyz="-0.08 -0.06 0.19"/>
+        <axis xyz="1 0 0"/>
+        <limit lower="-${PI/2}" upper="${PI/2}" effort="${effort}" velocity="${velocity}"/>
+        <mimic joint="arm_2_to_inner_circle" multiplier="-1" offset="0"/>
+        <dynamics damping="0.5" friction="0.1"/>
+    </joint>
+    <joint name="inner_circle_to_gripper_2" type="revolute">
+        <parent link="inner_circle"/>
+        <child link="gripper_2"/>
+        <origin rpy="0 0 0" xyz="-0.17 0.09 0.17"/>
+        <axis xyz="1 0 0"/>
+        <limit lower="-${PI/2}" upper="${PI/2}" effort="${effort}" velocity="${velocity}"/>
+        <mimic joint="arm_2_to_inner_circle" multiplier="-1" offset="0"/>
+        <dynamics damping="0.5" friction="0.1"/>
+    </joint>
+    <joint name="inner_circle_to_gripper_3" type="revolute">
+        <parent link="inner_circle"/>
+        <child link="gripper_3"/>
+        <origin rpy="0 0 ${4*PI/3}" xyz="-0.27 -0.04 0.16"/>
+        <axis xyz="1 0 0"/>
+        <limit lower="-${PI/2}" upper="${PI/2}" effort="${effort}" velocity="${velocity}"/>
+        <mimic joint="arm_2_to_inner_circle" multiplier="-1" offset="0"/>
+        <dynamics damping="0.5" friction="0.1"/>
+    </joint>
+</robot>

File: install/arduinobot_description/share/arduinobot_description/urdf/properties.xacro (robot description, xacro)
@@ -1 +1,12 @@
-/home/farr97/arduinobot_ws/src/arduinobot_description/urdf/properties.xacro
+<?xml version="1.0"?>
+<robot xmlns:xacro="http://www.ros.org/wiki/xacro">
+    <!-- Constants -->
+    <xacro:property name="PI" value="3.14159"/>
+    <xacro:property name="PI_2" value="${PI/2}"/>
+    <xacro:property name="PI_4" value="${PI/4}"/>
+    <!-- Joint properties -->
+    <xacro:property name="effort" value="30.0"/>
+    <xacro:property name="velocity" value="10.0"/>
+    <!-- Mark that properties are included -->
+    <xacro:property name="properties_included" value="1"/>
+</robot>
